File: Keyboard-schematics/schematic.kicad_pcb (KiCad board)
At the start: 2 copper layers, 44 x 44.1 mm, 25 parts, among them J1 USB_C_Receptacle_USB2.0, J2 Conn_01x05, U1 STM32F072CBT6, U2 PRTR5V0U2X, U3 XC6206PxxxMR-Regulator_Linear, U5 TXB0101

Commit message: PCB switch placement
Parts:
- added C10: 1uF, Capacitor_SMD:C_0402_1005Metric, F.Cu at (65.3, -63.7)
- added C2: 10uF, Capacitor_SMD:C_0603_1608Metric, F.Cu at (71.6, -59.5)
- added C43: 0.1uF, Capacitor_SMD:C_0402_1005Metric, F.Cu at (65.3, -61.7)
- added C44: 0.1uF, Capacitor_SMD:C_0402_1005Metric, F.Cu at (65.3, -59.8)
- added C8: 100nF, Capacitor_SMD:C_0402_1005Metric, F.Cu at (65.3, -67.7)
- added C9: 1uF, Capacitor_SMD:C_0402_1005Metric, F.Cu at (65.3, -65.7)
- added D1: D, Diode_SMD:D_SOD-123, B.Cu at (41.2, 38.5)
- added D10: D, Diode_SMD:D_SOD-123, B.Cu at (226.9, 38.5)
- added D11: D, Diode_SMD:D_SOD-123, B.Cu at (246.0, 38.5)
- added D12: D, Diode_SMD:D_SOD-123, B.Cu at (265.0, 38.5)
- added D13: D, Diode_SMD:D_SOD-123, B.Cu at (284.1, 38.5)
- added D14: D, Diode_SMD:D_SOD-123, B.Cu at (307.9, 38.5)
- added D15: D, Diode_SMD:D_SOD-123, B.Cu at (336.5, 38.5)
- added D16: D, Diode_SMD:D_SOD-123, B.Cu at (41.2, 62.3)
- added D17: D, Diode_SMD:D_SOD-123, B.Cu at (60.2, 62.3)
- added D18: D, Diode_SMD:D_SOD-123, B.Cu at (79.3, 62.3)
- added D19: D, Diode_SMD:D_SOD-123, B.Cu at (98.3, 62.3)
- added D2: D, Diode_SMD:D_SOD-123, B.Cu at (65.0, 38.5)
- added D20: D, Diode_SMD:D_SOD-123, B.Cu at (117.4, 62.3)
- added D21: D, Diode_SMD:D_SOD-123, B.Cu at (136.4, 62.3)
- added D22: D, Diode_SMD:D_SOD-123, B.Cu at (155.5, 62.3)
- added D23: D, Diode_SMD:D_SOD-123, B.Cu at (174.6, 62.3)
- added D24: D, Diode_SMD:D_SOD-123, B.Cu at (193.6, 62.3)
- added D25: D, Diode_SMD:D_SOD-123, B.Cu at (212.7, 62.3)
- added D26: D, Diode_SMD:D_SOD-123, B.Cu at (231.7, 62.3)
- added D27: D, Diode_SMD:D_SOD-123, B.Cu at (250.8, 62.3)
- added D28: D, Diode_SMD:D_SOD-123, B.Cu at (269.8, 62.3)
- added D29: D, Diode_SMD:D_SOD-123, B.Cu at (298.4, 62.3)
- added D3: D, Diode_SMD:D_SOD-123, B.Cu at (84.1, 38.5)
- added D30: D, Diode_SMD:D_SOD-123, B.Cu at (336.5, 62.3)
- added D31: D, Diode_SMD:D_SOD-123, B.Cu at (46.0, 81.3)
- added D32: D, Diode_SMD:D_SOD-123, B.Cu at (69.8, 81.3)
- added D33: D, Diode_SMD:D_SOD-123, B.Cu at (88.8, 81.3)
- added D34: D, Diode_SMD:D_SOD-123, B.Cu at (107.9, 81.3)
- added D35: D, Diode_SMD:D_SOD-123, B.Cu at (126.9, 81.3)
- added D36: D, Diode_SMD:D_SOD-123, B.Cu at (146.0, 81.3)
- added D37: D, Diode_SMD:D_SOD-123, B.Cu at (165.0, 81.3)
- added D38: D, Diode_SMD:D_SOD-123, B.Cu at (184.1, 81.3)
- added D39: D, Diode_SMD:D_SOD-123, B.Cu at (203.1, 81.3)
- added D4: D, Diode_SMD:D_SOD-123, B.Cu at (103.1, 38.5)
- added D40: D, Diode_SMD:D_SOD-123, B.Cu at (222.2, 81.3)
- added D41: D, Diode_SMD:D_SOD-123, B.Cu at (241.2, 81.3)
- added D42: D, Diode_SMD:D_SOD-123, B.Cu at (260.3, 81.3)
- added D43: D, Diode_SMD:D_SOD-123, B.Cu at (279.3, 81.3)
- added D44: D, Diode_SMD:D_SOD-123, B.Cu at (303.1, 81.3)
- added D45: D, Diode_SMD:D_SOD-123, B.Cu at (336.5, 81.3)
- added D46: D, Diode_SMD:D_SOD-123, B.Cu at (48.3, 100.4)
- added D47: D, Diode_SMD:D_SOD-123, B.Cu at (74.5, 100.4)
- added D48: D, Diode_SMD:D_SOD-123, B.Cu at (93.6, 100.4)
- added D49: D, Diode_SMD:D_SOD-123, B.Cu at (112.6, 100.4)
- added D5: D, Diode_SMD:D_SOD-123, B.Cu at (122.2, 38.5)
- added D50: D, Diode_SMD:D_SOD-123, B.Cu at (131.7, 100.4)
- added D51: D, Diode_SMD:D_SOD-123, B.Cu at (150.7, 100.4)
- added D52: D, Diode_SMD:D_SOD-123, B.Cu at (169.8, 100.4)
- added D53: D, Diode_SMD:D_SOD-123, B.Cu at (188.8, 100.4)
- added D54: D, Diode_SMD:D_SOD-123, B.Cu at (207.9, 100.4)
- added D55: D, Diode_SMD:D_SOD-123, B.Cu at (226.9, 100.4)
- added D56: D, Diode_SMD:D_SOD-123, B.Cu at (246.0, 100.4)
- added D57: D, Diode_SMD:D_SOD-123, B.Cu at (265.0, 100.4)
- added D58: D, Diode_SMD:D_SOD-123, B.Cu at (296.0, 100.4)
- added D59: D, Diode_SMD:D_SOD-123, B.Cu at (336.5, 100.4)
- added D6: D, Diode_SMD:D_SOD-123, B.Cu at (146.0, 38.5)
- added D60: D, Diode_SMD:D_SOD-123, B.Cu at (43.6, 119.4)
- added D61: D, Diode_SMD:D_SOD-123, B.Cu at (65.0, 119.4)
- added D62: D, Diode_SMD:D_SOD-123, B.Cu at (84.1, 119.4)
- added D63: D, Diode_SMD:D_SOD-123, B.Cu at (103.1, 119.4)
- added D64: D, Diode_SMD:D_SOD-123, B.Cu at (122.2, 119.4)
- added D65: D, Diode_SMD:D_SOD-123, B.Cu at (141.2, 119.4)
- added D66: D, Diode_SMD:D_SOD-123, B.Cu at (160.3, 119.4)
- added D67: D, Diode_SMD:D_SOD-123, B.Cu at (179.3, 119.4)
- added D68: D, Diode_SMD:D_SOD-123, B.Cu at (198.4, 119.4)
- added D69: D, Diode_SMD:D_SOD-123, B.Cu at (217.4, 119.4)
- added D7: D, Diode_SMD:D_SOD-123, B.Cu at (165.0, 38.5)
- added D70: D, Diode_SMD:D_SOD-123, B.Cu at (236.5, 119.4)
- added D71: D, Diode_SMD:D_SOD-123, B.Cu at (255.5, 119.4)
- added D72: D, Diode_SMD:D_SOD-123, B.Cu at (281.7, 119.4)
- added D73: D, Diode_SMD:D_SOD-123, B.Cu at (312.7, 124.2)
- added D74: D, Diode_SMD:D_SOD-123, B.Cu at (336.5, 119.4)
- added D75: D, Diode_SMD:D_SOD-123, B.Cu at (43.6, 143.2)
- added D76: D, Diode_SMD:D_SOD-123, B.Cu at (67.4, 143.2)
- added D77: D, Diode_SMD:D_SOD-123, B.Cu at (91.2, 143.2)
- added D78 (x2): D, Diode_SMD:D_SOD-123, B.Cu at (162.6, 143.2)
- added D79: D, Diode_SMD:D_SOD-123, B.Cu at (231.7, 143.2)
- added D8: D, Diode_SMD:D_SOD-123, B.Cu at (184.1, 38.5)
- added D80 (x2): D, Diode_SMD:D_SOD-123, B.Cu at (250.8, 143.2)
- added D81: D, Diode_SMD:D_SOD-123, B.Cu at (269.8, 143.2)
- added D82: D, Diode_SMD:D_SOD-123, B.Cu at (293.6, 143.2)
- added D83: D, Diode_SMD:D_SOD-123, B.Cu at (312.7, 143.2)
- added D84: D, Diode_SMD:D_SOD-123, B.Cu at (331.7, 143.2)
- added D9: D, Diode_SMD:D_SOD-123, B.Cu at (203.1, 38.5)
- added F1: 500mA, Fuse:Fuse_1206_3216Metric, F.Cu at (72.4, -62.4)
- added MX1: MX_SW_HS, PCM_marbastlib-mx:SW_MX_HS_CPG151101S11_1u, B.Cu at (38.1, 38.1)
- added MX10: MX_SW_HS, PCM_marbastlib-mx:SW_MX_HS_CPG151101S11_1u, B.Cu at (223.8, 38.1)
- added MX11: MX_SW_HS, PCM_marbastlib-mx:SW_MX_HS_CPG151101S11_1u, B.Cu at (242.9, 38.1)
- added MX12: MX_SW_HS, PCM_marbastlib-mx:SW_MX_HS_CPG151101S11_1u, B.Cu at (261.9, 38.1)
- added MX13: MX_SW_HS, PCM_marbastlib-mx:SW_MX_HS_CPG151101S11_1u, B.Cu at (281.0, 38.1)
- added MX14: MX_SW_HS, PCM_marbastlib-mx:SW_MX_HS_CPG151101S11_1u, B.Cu at (304.8, 38.1)
- added MX15: MX_SW_HS, PCM_marbastlib-mx:SW_MX_HS_CPG151101S11_1u, B.Cu at (333.4, 38.1)
- added MX16: MX_SW_HS, PCM_marbastlib-mx:SW_MX_HS_CPG151101S11_1u, B.Cu at (38.1, 61.9)
- added MX17: MX_SW_HS, PCM_marbastlib-mx:SW_MX_HS_CPG151101S11_1u, B.Cu at (57.1, 61.9)
- added MX18: MX_SW_HS, PCM_marbastlib-mx:SW_MX_HS_CPG151101S11_1u, B.Cu at (76.2, 61.9)
- added MX19: MX_SW_HS, PCM_marbastlib-mx:SW_MX_HS_CPG151101S11_1u, B.Cu at (95.2, 61.9)
- added MX2: MX_SW_HS, PCM_marbastlib-mx:SW_MX_HS_CPG151101S11_1u, B.Cu at (61.9, 38.1)
- added MX20: MX_SW_HS, PCM_marbastlib-mx:SW_MX_HS_CPG151101S11_1u, B.Cu at (114.3, 61.9)
- added MX21: MX_SW_HS, PCM_marbastlib-mx:SW_MX_HS_CPG151101S11_1u, B.Cu at (133.3, 61.9)
- added MX22: MX_SW_HS, PCM_marbastlib-mx:SW_MX_HS_CPG151101S11_1u, B.Cu at (152.4, 61.9)
- added MX23: MX_SW_HS, PCM_marbastlib-mx:SW_MX_HS_CPG151101S11_1u, B.Cu at (171.4, 61.9)
- added MX24: MX_SW_HS, PCM_marbastlib-mx:SW_MX_HS_CPG151101S11_1u, B.Cu at (190.5, 61.9)
- added MX25: MX_SW_HS, PCM_marbastlib-mx:SW_MX_HS_CPG151101S11_1u, B.Cu at (209.6, 61.9)
- added MX26: MX_SW_HS, PCM_marbastlib-mx:SW_MX_HS_CPG151101S11_1u, B.Cu at (228.6, 61.9)
- added MX27: MX_SW_HS, PCM_marbastlib-mx:SW_MX_HS_CPG151101S11_1u, B.Cu at (247.7, 61.9)
- added MX28: MX_SW_HS, PCM_marbastlib-mx:SW_MX_HS_CPG151101S11_1u, B.Cu at (266.7, 61.9)
- added MX29: MX_SW_HS, PCM_marbastlib-mx:SW_MX_HS_CPG151101S11_1u, B.Cu at (295.3, 61.9)
- added MX3: MX_SW_HS, PCM_marbastlib-mx:SW_MX_HS_CPG151101S11_1u, B.Cu at (81.0, 38.1)
- added MX30: MX_SW_HS, PCM_marbastlib-mx:SW_MX_HS_CPG151101S11_1u, B.Cu at (333.4, 61.9)
- added MX31: MX_SW_HS, PCM_marbastlib-mx:SW_MX_HS_CPG151101S11_1u, B.Cu at (42.9, 81.0)
- added MX32: MX_SW_HS, PCM_marbastlib-mx:SW_MX_HS_CPG151101S11_1u, B.Cu at (66.7, 81.0)
- added MX33: MX_SW_HS, PCM_marbastlib-mx:SW_MX_HS_CPG151101S11_1u, B.Cu at (85.7, 81.0)
- added MX34: MX_SW_HS, PCM_marbastlib-mx:SW_MX_HS_CPG151101S11_1u, B.Cu at (104.8, 81.0)
- added MX35: MX_SW_HS, PCM_marbastlib-mx:SW_MX_HS_CPG151101S11_1u, B.Cu at (123.8, 81.0)
- added MX36: MX_SW_HS, PCM_marbastlib-mx:SW_MX_HS_CPG151101S11_1u, B.Cu at (142.9, 81.0)
- added MX37: MX_SW_HS, PCM_marbastlib-mx:SW_MX_HS_CPG151101S11_1u, B.Cu at (161.9, 81.0)
- added MX38: MX_SW_HS, PCM_marbastlib-mx:SW_MX_HS_CPG151101S11_1u, B.Cu at (181.0, 81.0)
- added MX39: MX_SW_HS, PCM_marbastlib-mx:SW_MX_HS_CPG151101S11_1u, B.Cu at (200.0, 81.0)
- added MX4: MX_SW_HS, PCM_marbastlib-mx:SW_MX_HS_CPG151101S11_1u, B.Cu at (100.0, 38.1)
- added MX40: MX_SW_HS, PCM_marbastlib-mx:SW_MX_HS_CPG151101S11_1u, B.Cu at (219.1, 81.0)
- added MX41: MX_SW_HS, PCM_marbastlib-mx:SW_MX_HS_CPG151101S11_1u, B.Cu at (238.1, 81.0)
- added MX42: MX_SW_HS, PCM_marbastlib-mx:SW_MX_HS_CPG151101S11_1u, B.Cu at (257.2, 81.0)
- added MX43: MX_SW_HS, PCM_marbastlib-mx:SW_MX_HS_CPG151101S11_1u, B.Cu at (276.2, 81.0)
- added MX44: MX_SW_HS, PCM_marbastlib-mx:SW_MX_HS_CPG151101S11_1u, B.Cu at (300.0, 81.0)
- added MX45: MX_SW_HS, PCM_marbastlib-mx:SW_MX_HS_CPG151101S11_1u, B.Cu at (333.4, 81.0)
- added MX46: MX_SW_HS, PCM_marbastlib-mx:SW_MX_HS_CPG151101S11_1u, B.Cu at (45.2, 100.0)
- added MX47: MX_SW_HS, PCM_marbastlib-mx:SW_MX_HS_CPG151101S11_1u, B.Cu at (71.4, 100.0)
- added MX48: MX_SW_HS, PCM_marbastlib-mx:SW_MX_HS_CPG151101S11_1u, B.Cu at (90.5, 100.0)
- added MX49: MX_SW_HS, PCM_marbastlib-mx:SW_MX_HS_CPG151101S11_1u, B.Cu at (109.5, 100.0)
- added MX5: MX_SW_HS, PCM_marbastlib-mx:SW_MX_HS_CPG151101S11_1u, B.Cu at (119.1, 38.1)
- added MX50: MX_SW_HS, PCM_marbastlib-mx:SW_MX_HS_CPG151101S11_1u, B.Cu at (128.6, 100.0)
- added MX51: MX_SW_HS, PCM_marbastlib-mx:SW_MX_HS_CPG151101S11_1u, B.Cu at (147.6, 100.0)
- added MX52: MX_SW_HS, PCM_marbastlib-mx:SW_MX_HS_CPG151101S11_1u, B.Cu at (166.7, 100.0)
- added MX53: MX_SW_HS, PCM_marbastlib-mx:SW_MX_HS_CPG151101S11_1u, B.Cu at (185.7, 100.0)
- added MX54: MX_SW_HS, PCM_marbastlib-mx:SW_MX_HS_CPG151101S11_1u, B.Cu at (204.8, 100.0)
- added MX55: MX_SW_HS, PCM_marbastlib-mx:SW_MX_HS_CPG151101S11_1u, B.Cu at (223.8, 100.0)
- added MX56: MX_SW_HS, PCM_marbastlib-mx:SW_MX_HS_CPG151101S11_1u, B.Cu at (242.9, 100.0)
- added MX57: MX_SW_HS, PCM_marbastlib-mx:SW_MX_HS_CPG151101S11_1u, B.Cu at (261.9, 100.0)
- added MX58: MX_SW_HS, PCM_marbastlib-mx:SW_MX_HS_CPG151101S11_1u, B.Cu at (292.9, 100.0)
- added MX59: MX_SW_HS, PCM_marbastlib-mx:SW_MX_HS_CPG151101S11_1u, B.Cu at (333.4, 100.0)
- added MX6: MX_SW_HS, PCM_marbastlib-mx:SW_MX_HS_CPG151101S11_1u, B.Cu at (142.9, 38.1)
- added MX60: MX_SW_HS, PCM_marbastlib-mx:SW_MX_HS_CPG151101S11_1u, B.Cu at (40.5, 119.1)
- added MX61: MX_SW_HS, PCM_marbastlib-mx:SW_MX_HS_CPG151101S11_1u, B.Cu at (61.9, 119.1)
- added MX62: MX_SW_HS, PCM_marbastlib-mx:SW_MX_HS_CPG151101S11_1u, B.Cu at (81.0, 119.1)
- added MX63: MX_SW_HS, PCM_marbastlib-mx:SW_MX_HS_CPG151101S11_1u, B.Cu at (100.0, 119.1)
- added MX64: MX_SW_HS, PCM_marbastlib-mx:SW_MX_HS_CPG151101S11_1u, B.Cu at (119.1, 119.1)
- added MX65: MX_SW_HS, PCM_marbastlib-mx:SW_MX_HS_CPG151101S11_1u, B.Cu at (138.1, 119.1)
- added MX66: MX_SW_HS, PCM_marbastlib-mx:SW_MX_HS_CPG151101S11_1u, B.Cu at (157.2, 119.1)
- added MX67: MX_SW_HS, PCM_marbastlib-mx:SW_MX_HS_CPG151101S11_1u, B.Cu at (176.2, 119.1)
- added MX68: MX_SW_HS, PCM_marbastlib-mx:SW_MX_HS_CPG151101S11_1u, B.Cu at (195.3, 119.1)
- added MX69: MX_SW_HS, PCM_marbastlib-mx:SW_MX_HS_CPG151101S11_1u, B.Cu at (214.3, 119.1)
- added MX7: MX_SW_HS, PCM_marbastlib-mx:SW_MX_HS_CPG151101S11_1u, B.Cu at (161.9, 38.1)
- added MX70: MX_SW_HS, PCM_marbastlib-mx:SW_MX_HS_CPG151101S11_1u, B.Cu at (233.4, 119.1)
- added MX71: MX_SW_HS, PCM_marbastlib-mx:SW_MX_HS_CPG151101S11_1u, B.Cu at (252.4, 119.1)
- added MX72: MX_SW_HS, PCM_marbastlib-mx:SW_MX_HS_CPG151101S11_1u, B.Cu at (278.6, 119.1)
- added MX73: MX_SW_HS, PCM_marbastlib-mx:SW_MX_HS_CPG151101S11_1u, B.Cu at (309.6, 123.8)
- added MX74: MX_SW_HS, PCM_marbastlib-mx:SW_MX_HS_CPG151101S11_1u, B.Cu at (333.4, 119.1)
- added MX75: MX_SW_HS, PCM_marbastlib-mx:SW_MX_HS_CPG151101S11_1u, B.Cu at (40.5, 142.9)
- added MX76: MX_SW_HS, PCM_marbastlib-mx:SW_MX_HS_CPG151101S11_1u, B.Cu at (64.3, 142.9)
- added MX77: MX_SW_HS, PCM_marbastlib-mx:SW_MX_HS_CPG151101S11_1u, B.Cu at (88.1, 142.9)
- added MX78: MX_SW_HS, PCM_marbastlib-mx:SW_MX_HS_CPG151101S11_1u, B.Cu at (159.5, 142.9)
- added MX79: MX_SW_HS, PCM_marbastlib-mx:SW_MX_HS_CPG151101S11_1u, B.Cu at (228.6, 142.9)
- added MX8: MX_SW_HS, PCM_marbastlib-mx:SW_MX_HS_CPG151101S11_1u, B.Cu at (181.0, 38.1)
- added MX80 (x2): MX_SW_HS, PCM_marbastlib-mx:SW_MX_HS_CPG151101S11_1u, B.Cu at (247.7, 142.9)
- added MX81: MX_SW_HS, PCM_marbastlib-mx:SW_MX_HS_CPG151101S11_1u, B.Cu at (266.7, 142.9)
- added MX82: MX_SW_HS, PCM_marbastlib-mx:SW_MX_HS_CPG151101S11_1u, B.Cu at (290.5, 142.9)
- added MX83: MX_SW_HS, PCM_marbastlib-mx:SW_MX_HS_CPG151101S11_1u, B.Cu at (309.6, 142.9)
- added MX84: MX_SW_HS, PCM_marbastlib-mx:SW_MX_HS_CPG151101S11_1u, B.Cu at (328.6, 142.9)
- added MX9: MX_SW_HS, PCM_marbastlib-mx:SW_MX_HS_CPG151101S11_1u, B.Cu at (200.0, 38.1)
- added R1: 5.1k, Resistor_SMD:R_0402_1005Metric, F.Cu at (68.2, -63.0)
- added R2: 5.1k, Resistor_SMD:R_0402_1005Metric, F.Cu at (68.2, -61.0)
- added U2: PRTR5V0U2X, Package_TO_SOT_SMD:SOT-143, F.Cu at (68.8, -66.2)
- added U3: XC6206PxxxMR-Regulator_Linear, Package_TO_SOT_SMD:SOT-23, F.Cu at (73.4, -66.4)
- moved C4 246.2 mm to (411.9, -50.1)
- moved C43 246.2 mm to (406.4, -54.7)
- moved C7 246.2 mm to (406.5, -40.4)
- moved F1 246.2 mm to (412.5, -53.4)
- moved R4 246.2 mm to (433.6, -37.2)
- moved U5 246.2 mm to (404.9, -52.7)
- moved BOOT1 246.2 mm to (434.3, -31.7)
- moved C1 246.2 mm to (405.6, -39.5)
- moved C10 246.2 mm to (401.8, -43.7)
- moved C2 246.2 mm to (401.9, -42.5)
- moved C44 246.2 mm to (403.4, -54.7)
- moved C5 246.2 mm to (412.3, -37.7)
- moved C8 246.2 mm to (426.2, -44.5)
- moved C9 246.2 mm to (399.2, -46.5)
- moved J1 246.2 mm to (423.7, -53.9)
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Routing:
- net +5V: track 10.3 -> 4.57 mm, vias 4 -> 0
- net Net-(D84-A): track 0.00 -> 4.01 mm
- net Net-(D83-A): track 0.00 -> 4.01 mm
- net Net-(D82-A): track 0.00 -> 4.01 mm
- net Net-(D81-A): track 0.00 -> 4.01 mm
- net Net-(D80-A): track 0.00 -> 4.01 mm
- net Net-(D79-A): track 0.00 -> 4.01 mm
- net Net-(D78-A): track 0.00 -> 4.01 mm
- net Net-(D77-A): track 0.00 -> 4.01 mm
- net Net-(D76-A): track 0.00 -> 4.01 mm
- net Net-(D74-A): track 0.00 -> 4.01 mm
- net Net-(D73-A): track 0.00 -> 4.01 mm
- net Net-(D72-A): track 0.00 -> 4.01 mm
- net Net-(D71-A): track 0.00 -> 4.01 mm
- net Net-(D70-A): track 0.00 -> 4.01 mm
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
Commit message: Switch wire routing
Parts:
- removed the MX80 at (247.7, 142.9)
Routing:
- net row_4: track 0.00 -> 300.8 mm
- net row_1: track 0.00 -> 299.5 mm
- net row_2: track 0.00 -> 294.6 mm
- net row_3: track 0.00 -> 292.0 mm
- net row_5: track 0.00 -> 290.9 mm
- net row_0: track 0.00 -> 270.7 mm
- net col_11: track 0.00 -> 126.5 mm
- net col_9: track 0.00 -> 126.5 mm
- net col_10: track 0.00 -> 126.5 mm
- net col_13: track 0.00 -> 120.6 mm
- net col_12: track 0.00 -> 120.6 mm
- net col_6: track 0.00 -> 119.6 mm
- net col_2: track 0.00 -> 119.6 mm
- net col_1: track 0.00 -> 117.6 mm
- net col_0: track 0.00 -> 109.7 mm
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
Commit message: Alternative layout wiring
Parts:
- removed the C10 at (65.3, -63.7)
- removed the C10 at (401.8, -43.7)
- removed the C2 at (71.6, -59.5)
- removed the C2 at (401.9, -42.5)
- removed the C43 at (65.3, -61.7)
- removed the C43 at (406.4, -54.7)
- removed the C44 at (65.3, -59.8)
- removed the C44 at (403.4, -54.7)
- removed the C8 at (65.3, -67.7)
- removed the C8 at (426.2, -44.5)
- removed the C9 at (65.3, -65.7)
- removed the C9 at (399.2, -46.5)
- removed the F1 at (72.4, -62.4)
- removed the F1 at (412.5, -53.4)
- removed the R1 at (68.2, -63.0)
- removed the R1 at (427.7, -46.0)
- removed the R2 at (68.2, -61.0)
- removed the R2 at (426.7, -47.2)
- removed the U2 at (68.8, -66.2)
- removed the U2 at (423.7, -45.9)
- removed the U3 at (73.4, -66.4)
- removed the U3 at (401.7, -46.0)
- added C10: 1uF, Capacitor_SMD:C_0402_1005Metric, B.Cu at (360.4, 32.1)
- added C2: 10uF, Capacitor_SMD:C_0603_1608Metric, B.Cu at (360.6, 33.3)
- added C43: 0.1uF, Capacitor_SMD:C_0402_1005Metric, B.Cu at (365.0, 21.1)
- added C44: 0.1uF, Capacitor_SMD:C_0402_1005Metric, B.Cu at (362.0, 21.1)
- added C8: 100nF, Capacitor_SMD:C_0402_1005Metric, B.Cu at (384.9, 31.3)
- added C9: 1uF, Capacitor_SMD:C_0402_1005Metric, B.Cu at (357.8, 29.3)
- added D29_alt1: D, Diode_SMD:D_SOD-123, B.Cu at (274.6, 100.4)
- added F1: 500mA, Fuse:Fuse_1206_3216Metric, B.Cu at (371.1, 22.4)
- added MX29_alt1: MX_SW_HS, PCM_marbastlib-mx:SW_MX_HS_CPG151101S11_1u, B.Cu at (285.8, 61.9)
- added MX29_alt2: MX_SW_HS, PCM_marbastlib-mx:SW_MX_HS_CPG151101S11_1u, B.Cu at (304.8, 61.9)
- added MX46_alt1: MX_SW_HS, PCM_marbastlib-mx:SW_MX_HS_CPG151101S11_1u, B.Cu at (38.1, 100.0)
- added MX60_alt1: MX_SW_HS, PCM_marbastlib-mx:SW_MX_HS_CPG151101S11_1u, B.Cu at (50.0, 119.1)
- added MX78: MX_SW_HS, PCM_marbastlib-mx:SW_MX_HS_CPG151101S11_1u, B.Cu at (119.1, 142.9)
- added MX80: MX_SW_HS, PCM_marbastlib-mx:SW_MX_HS_CPG151101S11_1u, B.Cu at (200.0, 142.9)
- added R1: 5.1k, Resistor_SMD:R_0402_1005Metric, B.Cu at (386.3, 29.8)
- added R2: 5.1k, Resistor_SMD:R_0402_1005Metric, B.Cu at (385.3, 28.6)
- added S1: MX_stab, PCM_marbastlib-mx:STAB_MX_P_2u, F.Cu at (295.3, 61.9)
- added S2: MX_stab, PCM_marbastlib-mx:STAB_MX_P_2.25u, F.Cu at (292.9, 100.0)
- added S3: MX_stab, PCM_marbastlib-mx:STAB_MX_P_2.25u, F.Cu at (50.0, 119.1)
- added S4: MX_stab, PCM_marbastlib-mx:STAB_MX_P_2u, F.Cu at (119.1, 142.9)
- added S5: MX_stab, PCM_marbastlib-mx:STAB_MX_P_2.25u, F.Cu at (159.5, 142.9)
- added S6: MX_stab, PCM_marbastlib-mx:STAB_MX_P_2u, F.Cu at (200.0, 142.9)
- added S7: MX_stab, PCM_marbastlib-mx:STAB_MX_P_6.25u, F.Cu at (159.5, 142.9)
- added U2: PRTR5V0U2X, Package_TO_SOT_SMD:SOT-143, B.Cu at (382.3, 29.9)
- added U3: XC6206PxxxMR-Regulator_Linear, Package_TO_SOT_SMD:SOT-23, B.Cu at (360.3, 29.8)
- U5: footprint Package_TO_SOT_SMD:SOT-363_SC-70-6_Handsoldering -> Package_TO_SOT_SMD:SOT-363_SC-70-6
- moved C1 86.3 mm to (364.2, 36.3)
- moved C5 86.3 mm to (370.9, 38.1)
- moved C7 86.3 mm to (365.1, 35.4)
- moved J1 86.3 mm to (382.3, 21.9)
- moved J2 86.3 mm to (392.1, 22.8)
- moved R4 86.3 mm to (392.2, 38.6)
- moved U5 86.3 mm to (363.5, 23.1)
- moved BOOT1 86.3 mm to (392.9, 44.1)
- moved C4 86.3 mm to (370.6, 25.7)
- moved C3 86.3 mm to (376.9, 31.7)
- moved C6 86.3 mm to (369.5, 38.8)
- moved R3 86.3 mm to (391.0, 38.7)
- moved RST1 86.3 mm to (393.0, 55.3)
- moved U1 86.3 mm to (370.8, 31.9)
- moved D80 47.6 mm to (203.1, 143.2)
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- renumbered D74 to D73, D73 to D74, D78 to D79, D79 to D81, D80 to D82, D81 to D83, D82 to D84, D83 to D85, D84 to D86, MX74 to MX73, MX73 to MX74, MX78 to MX79, MX79 to MX81, MX80 to MX82, MX81 to MX83, MX82 to MX84, MX83 to MX85, MX84 to MX86
Connections:
- D79 pad 2: Net-(D78-A) -> Net-(D79-A)
- D82 pad 2: Net-(D80-A) -> Net-(D82-A)
- MX79 pad 2: Net-(D78-A) -> Net-(D79-A)
- MX82 pad 2: Net-(D80-A) -> Net-(D82-A)
Routing:
- net GND: track 119.2 -> 184.0 mm, vias 4 -> 9
- net Net-(D29_alt1-A): track 0.00 -> 47.5 mm, vias 0 -> 1
- net +5V: track 4.57 -> 40.5 mm, vias 0 -> 2
- net col_0: track 109.7 -> 143.3 mm
- net col_8: track 94.8 -> 120.6 mm
- net row_0: track 270.7 -> 296.4 mm
- net Net-(D29-A): track 4.01 -> 28.9 mm
- net col_4: track 92.8 -> 116.6 mm
- net Net-(D46-A): track 4.01 -> 24.6 mm
- net Net-(D60-A): track 4.01 -> 22.7 mm
- net row_3: track 292.0 -> 274.5 mm
- net row_4: track 300.8 -> 286.1 mm
- net col_12: track 120.6 -> 133.7 mm
- net row_2: track 294.6 -> 282.8 mm
- net row_5: track 290.9 -> 284.9 mm
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Other:
- board size 44 x 44.1 mm -> 377.8 x 142.9 mm
