File: Keyboard-schematics/switches.kicad_sch (KiCad schematic)
At the start: 175 parts

Commit message: Assigned footprints to diodes
Parts:
- D1, D10, D11, D12, D13, D14, D15, D16, D17, D18, D19, D2, D20, D21, D22, D23, D24, D25, D26, D27, D28, D29, D3, D30, D31, D32, D33, D34, D35, D36, D37, D38, D39, D4, D40, D41, D42, D43, D44, D45, D46, D47, D48, D49, D5, D50, D51, D52, D53, D54, D55, D56, D57, D58, D59, D6, D60, D61, D62, D63, D64, D65, D66, D67, D68, D69, D7, D70, D71, D72, D73, D74, D75, D76, D77, D8, D9: footprint (none) -> Diode_SMD:D_SOD-123
- D78: renamed from D85; footprint (none) -> Diode_SMD:D_SOD-123
- D79: renamed from D86; footprint (none) -> Diode_SMD:D_SOD-123
- D80: renamed from D78; footprint (none) -> Diode_SMD:D_SOD-123
- D81: renamed from D79; footprint (none) -> Diode_SMD:D_SOD-123
- D82: renamed from D80; footprint (none) -> Diode_SMD:D_SOD-123
- D83: renamed from D81; footprint (none) -> Diode_SMD:D_SOD-123
- D84: renamed from D82; footprint (none) -> Diode_SMD:D_SOD-123
- D85: renamed from D83; footprint (none) -> Diode_SMD:D_SOD-123
- D86: renamed from D84; footprint (none) -> Diode_SMD:D_SOD-123
- renumbered MX28_alt to MX28_alt1, MX46_alt to MX46_alt1, MX60_alt to MX60_alt1, MX85 to MX78, MX86 to MX79, MX78 to MX80, MX79 to MX81, MX80 to MX82, MX81 to MX83, MX82 to MX84, MX83 to MX85, MX84 to MX86
Connections:
- net row_5: now also D78.1 (K), D79.1 (K)
Other:
- moved on the sheet: D78, D79, MX78, MX79

Commit message: PCB switch placement
Parts:
- removed D78, D80: D, Diode_SMD:D_SOD-123, symbol Device:D
- removed MX28_alt1, MX46_alt1, MX60_alt1, MX78, MX80: MX_SW_HS, PCM_marbastlib-mx:SW_MX_HS_CPG151101S11_1u, symbol PCM_marbastlib-mx:MX_SW_HS_CPG151101S11
- renumbered D74 to D73, D73 to D74, D79 to D78, D81 to D79, D82 to D80, D83 to D81, D84 to D82, D85 to D83, D86 to D84, MX74 to MX73, MX73 to MX74, MX79 to MX78, MX81 to MX79, MX82 to MX80, MX83 to MX81, MX84 to MX82, MX85 to MX83, MX86 to MX84
Connections:
- net col_13: now also MX73.1; no longer MX74.1
- net col_14: now also MX74.1; no longer MX73.1
Other:
- moved on the sheet: D73, D74, MX73, MX74

Commit message: Alternative layout wiring
Parts:
- added D29_alt1, D78, D80: D, Diode_SMD:D_SOD-123, symbol Device:D
- added MX29_alt1, MX29_alt2, MX46_alt1, MX60_alt1, MX78, MX80: MX_SW_HS, PCM_marbastlib-mx:SW_MX_HS_CPG151101S11_1u, symbol PCM_marbastlib-mx:MX_SW_HS_CPG151101S11
- added S1, S4, S6: MX_stab, PCM_marbastlib-mx:STAB_MX_P_2u, symbol PCM_marbastlib-mx:MX_stab
- added S2, S3, S5: MX_stab, PCM_marbastlib-mx:STAB_MX_P_2.25u, symbol PCM_marbastlib-mx:MX_stab
- added S7: MX_stab, PCM_marbastlib-mx:STAB_MX_P_6.25u, symbol PCM_marbastlib-mx:MX_stab
- renumbered D78 to D79, D79 to D81, D80 to D82, D81 to D83, D82 to D84, D83 to D85, D84 to D86, MX78 to MX79, MX79 to MX81, MX80 to MX82, MX81 to MX83, MX82 to MX84, MX83 to MX85, MX84 to MX86
Connections:
- net col_0: now also MX46_alt1.1, MX60_alt1.1
- net col_12: now also MX29_alt1.1
- net col_13: now also MX74.1, MX29_alt2.1; no longer MX73.1
- net col_14: now also MX73.1; no longer MX74.1
- net col_4: now also MX78.1
- net col_8: now also MX80.1
- net row_3: now also D29_alt1.1 (K)
- net row_5: now also D78.1 (K), D80.1 (K)
- net at D46.2 (A), MX46.2: now also MX46_alt1.2
- net at D29.2 (A), MX29.2: now also MX29_alt2.2
- net at D60.2 (A), MX60.2: now also MX60_alt1.2
- new net: D80.2 (A), MX80.2
- new net: D29_alt1.2 (A), MX29_alt1.2
- new net: D78.2 (A), MX78.2
Other:
- moved on the sheet: D73, D74, MX73, MX74
