File: 96%/switches.kicad_sch (KiCad schematic)
At the start: 212 parts

Commit message: LED wiring for 96% layout
Parts:
- S67: footprint PCM_marbastlib-mx:STAB_MX_P_2u -> PCM_marbastlib-mx:STAB_MX_P_2.25u
Changed lines of the file:
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@@
 			)
 		)
-		(property "Footprint" "PCM_marbastlib-mx:STAB_MX_P_2u"
+		(property "Footprint" "PCM_marbastlib-mx:STAB_MX_P_2.25u"
 			(at 274.32 35.56 0)
 			(effects
