File: 96%/led_backlight.kicad_sch (KiCad schematic)
At the start: 98 parts

Commit message: Finished LEDs wirign
Parts:
- LED1, LED10, LED100, LED11, LED12, LED13, LED14, LED15, LED16, LED17, LED18, LED19, LED2, LED20, LED21, LED22, LED23, LED24, LED25, LED26, LED27, LED28, LED29, LED3, LED31, LED32, LED33, LED34, LED35, LED36, LED37, LED38, LED39, LED4, LED40, LED41, LED42, LED43, LED44, LED45, LED46, LED47, LED48, LED49, LED5, LED50, LED51, LED52, LED53, LED54, LED55, LED56, LED57, LED58, LED59, LED6, LED60, LED61, LED62, LED63, LED64, LED65, LED66, LED67, LED68, LED69, LED7, LED71, LED72, LED73, LED74, LED75, LED76, LED77, LED78, LED79, LED8, LED80, LED81, LED82, LED83, LED84, LED85, LED86, LED87, LED88, LED89, LED9, LED90, LED91, LED92, LED93, LED94, LED95, LED96, LED97, LED98, LED99: footprint PCM_marbastlib-various:LED_6028R_no_cutout -> PCM_marbastlib-various:LED_6028R

Commit message: Finished wiring on 96% keyboard
Parts:
- added C100, C101, C102, C103, C104, C105, C106, C107, C108, C109, C110, C13, C14, C15, C16, C17, C18, C19, C20, C21, C22, C23, C24, C25, C26, C27, C28, C29, C30, C31, C32, C33, C34, C35, C36, C37, C38, C39, C40, C41, C42, C43, C44, C45, C46, C47, C48, C49, C50, C51, C52, C53, C54, C55, C56, C57, C58, C59, C60, C61, C62, C63, C64, C65, C66, C67, C68, C69, C70, C71, C72, C73, C74, C75, C76, C77, C78, C79, C80, C81, C82, C83, C84, C85, C86, C87, C88, C89, C90, C91, C92, C93, C94, C95, C96, C97, C98, C99: 100nF, Capacitor_SMD:C_0402_1005Metric, symbol Device:C
- added R5: 500OHM, Resistor_SMD:R_0402_1005Metric, symbol Device:R
- added ULED1, ULED10, ULED11, ULED12, ULED13, ULED14, ULED15, ULED16, ULED17, ULED18, ULED19, ULED2, ULED20, ULED3, ULED4, ULED5, ULED6, ULED7, ULED8, ULED9: WS2812B-2020, LED_SMD:LED_WS2812B-2020_PLCC4_2.0x2.0mm, symbol LED:WS2812B-2020
- renumbered LED31 to LED30, LED32 to LED31, LED33 to LED32, LED34 to LED33, LED35 to LED34, LED36 to LED35, LED37 to LED36, LED38 to LED37, LED39 to LED38, LED40 to LED39, LED41 to LED40, LED42 to LED41, LED43 to LED42, LED44 to LED43, LED45 to LED44, LED46 to LED45, LED47 to LED46, LED48 to LED47, LED49 to LED48, LED50 to LED49, LED51 to LED50, LED52 to LED51, LED53 to LED52, LED54 to LED53, LED55 to LED54, LED56 to LED55, LED57 to LED56, LED58 to LED57, LED59 to LED58, LED60 to LED59, LED61 to LED60, LED62 to LED61, LED63 to LED62, LED64 to LED63, LED65 to LED64, LED66 to LED65, LED67 to LED66, LED68 to LED67, LED69 to LED68, LED71 to LED69, LED72 to LED70, LED73 to LED71, LED74 to LED72, LED75 to LED73, LED76 to LED74, LED77 to LED75, LED78 to LED76, LED79 to LED77, LED80 to LED78, LED81 to LED79, LED85 to LED80, LED82 to LED81, LED83 to LED82, LED84 to LED83, LED86 to LED84, LED87 to LED85, LED88 to LED86, LED89 to LED87, LED90 to LED88, LED91 to LED89, LED92 to LED90, LED93 to LED91, LED94 to LED92, LED95 to LED93, LED98 to LED94, LED99 to LED95, LED100 to LED96, LED96 to LED97, LED97 to LED98
Connections:
- net GND: now also C100.1, C101.1, C102.1, C103.1, C104.1, C105.1, C106.1, C107.1, C108.1, C109.1, C110.1, C13.1, C14.1, C15.1, C16.1, C17.1, C18.1, C19.1, C20.1, C21.1, C22.1, C23.1, C24.1, C25.1, C26.1, C27.1, C28.1, C29.1, C30.1, C31.1, C32.1, C33.1, C34.1, C35.1, C36.1, C37.1, C38.1, C39.1, C40.1, C41.1, C42.1, C43.1, C44.1, C45.1, C46.1, C47.1, C48.1, C49.1, C50.1, C51.1, C52.1, C53.1, C54.1, C55.1, C56.1, C57.1, C58.1, C59.1, C60.1, C61.1, C62.1, C63.1, C64.1, C65.1, C66.1, C67.1, C68.1, C69.1, C70.1, C71.1, C72.1, C73.1, C74.1, C75.1, C76.1, C77.1, C78.1, C79.1, C80.1, C81.1, C82.1, C83.1, C84.1, C85.1, C86.1, C87.1, C88.1, C89.1, C90.1, C91.1, C92.1, C93.1, C94.1, C95.1, C96.1, C97.1, C98.1, C99.1, ULED1.2 (VSS), ULED10.2 (VSS), ULED11.2 (VSS), ULED12.2 (VSS), ULED13.2 (VSS), ULED14.2 (VSS), ULED15.2 (VSS), ULED16.2 (VSS), ULED17.2 (VSS), ULED18.2 (VSS), ULED19.2 (VSS), ULED2.2 (VSS), ULED20.2 (VSS), ULED3.2 (VSS), ULED4.2 (VSS), ULED5.2 (VSS), ULED6.2 (VSS), ULED7.2 (VSS), ULED8.2 (VSS), ULED9.2 (VSS)
- net VDD: now also C100.2, C101.2, C102.2, C103.2, C104.2, C105.2, C106.2, C107.2, C108.2, C109.2, C110.2, C13.2, C14.2, C15.2, C16.2, C17.2, C18.2, C19.2, C20.2, C21.2, C22.2, C23.2, C24.2, C25.2, C26.2, C27.2, C28.2, C29.2, C30.2, C31.2, C32.2, C33.2, C34.2, C35.2, C36.2, C37.2, C38.2, C39.2, C40.2, C41.2, C42.2, C43.2, C44.2, C45.2, C46.2, C47.2, C48.2, C49.2, C50.2, C51.2, C52.2, C53.2, C54.2, C55.2, C56.2, C57.2, C58.2, C59.2, C60.2, C61.2, C62.2, C63.2, C64.2, C65.2, C66.2, C67.2, C68.2, C69.2, C70.2, C71.2, C72.2, C73.2, C74.2, C75.2, C76.2, C77.2, C78.2, C79.2, C80.2, C81.2, C82.2, C83.2, C84.2, C85.2, C86.2, C87.2, C88.2, C89.2, C90.2, C91.2, C92.2, C93.2, C94.2, C95.2, C96.2, C97.2, C98.2, C99.2, ULED1.4 (VDD), ULED10.4 (VDD), ULED11.4 (VDD), ULED12.4 (VDD), ULED13.4 (VDD), ULED14.4 (VDD), ULED15.4 (VDD), ULED16.4 (VDD), ULED17.4 (VDD), ULED18.4 (VDD), ULED19.4 (VDD), ULED2.4 (VDD), ULED20.4 (VDD), ULED3.4 (VDD), ULED4.4 (VDD), ULED5.4 (VDD), ULED6.4 (VDD), ULED7.4 (VDD), ULED8.4 (VDD), ULED9.4 (VDD)
- net led_input: now also R5.2; no longer LED15.3 (DIN)
- net at LED74.2 (DOUT): now also ULED15.3 (DIN); no longer LED73.3 (DIN)
- net at LED34.3 (DIN): now also ULED10.1 (DOUT); no longer LED35.2 (DOUT)
- net at LED8.2 (DOUT): now also ULED4.3 (DIN); no longer LED7.3 (DIN)
- net at LED70.2 (DOUT): now also ULED13.3 (DIN); no longer LED69.3 (DIN)
- net at LED50.3 (DIN): now also ULED11.1 (DOUT); no longer LED51.2 (DOUT)
- net at LED84.2 (DOUT): now also ULED20.3 (DIN); no longer LED83.3 (DIN)
- net at LED75.3 (DIN): now also ULED16.1 (DOUT); no longer LED76.2 (DOUT)
- net at LED9.3 (DIN): now also ULED5.1 (DOUT); no longer LED10.2 (DOUT)
- net at LED69.2 (DOUT): now also ULED12.3 (DIN); no longer LED68.3 (DIN)
- net at LED71.3 (DIN): now also ULED14.1 (DOUT); no longer LED72.2 (DOUT)
- net at LED3.3 (DIN): now also ULED2.1 (DOUT); no longer LED4.2 (DOUT)
- net at LED81.3 (DIN): now also ULED19.1 (DOUT); no longer LED82.2 (DOUT)
- net at LED80.2 (DOUT): now also ULED18.3 (DIN); no longer LED79.3 (DIN)
- net at LED11.3 (DIN): now also ULED6.1 (DOUT); no longer LED12.2 (DOUT)
- net at LED5.3 (DIN): now also ULED3.1 (DOUT); no longer LED6.2 (DOUT)
- net at LED77.3 (DIN): now also ULED17.1 (DOUT); no longer LED78.2 (DOUT)
- net at LED1.3 (DIN): now also ULED1.1 (DOUT); no longer LED2.2 (DOUT)
- net at LED13.3 (DIN): now also ULED7.1 (DOUT); no longer LED14.2 (DOUT)
- net led_output: no longer names the net of LED98.2 (DOUT)
- new net: LED6.2 (DOUT), ULED3.3 (DIN)
- new net: R5.1, ULED9.3 (DIN)
- new net: LED72.2 (DOUT), ULED14.3 (DIN)
- new net: LED4.2 (DOUT), ULED2.3 (DIN)
- new net: LED35.2 (DOUT), ULED10.3 (DIN)
- new net: LED69.3 (DIN), ULED13.1 (DOUT)
- new net: LED73.3 (DIN), ULED15.1 (DOUT)
- new net: LED15.3 (DIN), ULED8.1 (DOUT)
- new net: ULED8.3 (DIN), ULED9.1 (DOUT)
- new net: LED68.3 (DIN), ULED12.1 (DOUT)
- new net: LED82.2 (DOUT), ULED19.3 (DIN)
- new net: LED10.2 (DOUT), ULED5.3 (DIN)
- new net: LED76.2 (DOUT), ULED16.3 (DIN)
- new net: LED12.2 (DOUT), ULED6.3 (DIN)
- new net: LED7.3 (DIN), ULED4.1 (DOUT)
- new net: LED2.2 (DOUT), ULED1.3 (DIN)
- new net: LED79.3 (DIN), ULED18.1 (DOUT)
- new net: LED78.2 (DOUT), ULED17.3 (DIN)
- new net: LED51.2 (DOUT), ULED11.3 (DIN)
- new net: LED83.3 (DIN), ULED20.1 (DOUT)
- new net: LED14.2 (DOUT), ULED7.3 (DIN)
- no-connect marks 0 -> 1
Other:
- moved on the sheet: LED1, LED10, LED11, LED12, LED13, LED14, LED15, LED16, LED17, LED18, LED19, LED2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
